File: nRF24-module.sch (KiCad schematic (older format))
At the start: 29 parts, among them P1 CONN_02X04, U1 STM32F302C8T, U2 SN65HVD256, U3 MCP1703, X1 16MHz 10ppm

Commit message: Change LED polarity, optimize routing
Parts:
- C1, C10, C11, C12, C13, C2, C3, C4, C5, C6, C7, C8, C9: footprint _std:_0603 -> Capacitors_SMD:C_0603
- D1, D2: footprint _std:_0603 -> LEDs:LED-0603
- R2, R3, R4: footprint _std:_0603 -> Resistors_SMD:R_0603
- U3: footprint _std:_SOT23-3 -> _div:_MCP1703-SOT-23A
Connections:
- net GND: now also D1.1 (K), D2.1 (K)
- net RX_LED: now also R2.1; no longer D1.1 (K)
- net TX_LED: now also R3.1; no longer D2.1 (K)
- net VCC: no longer R2.2, R3.2
- net at D2.2 (A): now also R3.2; no longer R3.1
- net at D1.2 (A): now also R2.2; no longer R2.1
Other:
- note removed: "04.11.2015"
- note removed: "A"
- note removed: "Author: Michael Spieler"
- note removed: "nRF24 radio module"
- moved on the sheet: D1, D2, R2, R3
Changed lines of the file:
@@
 encoding utf-8
 Sheet 1 1
-Title ""
-Date ""
-Rev ""
-Comp ""
+Title "nRF24 CAN radio module"
+Date "2016-06-05"
+Rev "A"
+Comp "Author: Michael Spieler"
 Comment1 ""
 Comment2 ""
@@
 F 0 "C5" H 1825 2450 50  0000 L CNN
 F 1 "100nF" H 1825 2250 50  0000 L CNN
-F 2 "_std:_0603" H 1838 2200 30  0001 C CNN
+F 2 "Capacitors_SMD:C_0603" H 1838 2200 30  0001 C CNN
 F 3 "" H 1800 2350 60  0000 C CNN
 	1    1800 2350
@@
 F 0 "C3" H 1575 2450 50  0000 L CNN
 F 1 "100nF" H 1575 2250 50  0000 L CNN
-F 2 "_std:_0603" H 1588 2200 30  0001 C CNN
+F 2 "Capacitors_SMD:C_0603" H 1588 2200 30  0001 C CNN
 F 3 "" H 1550 2350 60  0000 C CNN
 	1    1550 2350
@@
 F 0 "C2" H 1325 2450 50  0000 L CNN
 F 1 "100nF" H 1325 2250 50  0000 L CNN
-F 2 "_std:_0603" H 1338 2200 30  0001 C CNN
+F 2 "Capacitors_SMD:C_0603" H 1338 2200 30  0001 C CNN
 F 3 "" H 1300 2350 60  0000 C CNN
 	1    1300 2350
@@
 F 0 "C1" H 1075 2450 50  0000 L CNN
 F 1 "4.7uF" H 1075 2250 50  0000 L CNN
-F 2 "_std:_0603" H 1088 2200 30  0001 C CNN
+F 2 "Capacitors_SMD:C_0603" H 1088 2200 30  0001 C CNN
 F 3 "" H 1050 2350 60  0000 C CNN
 	1    1050 2350
@@
 F 0 "C7" H 4375 5700 50  0000 L CNN
 F 1 "10pF" H 4150 5500 50  0000 L CNN
-F 2 "_std:_0603" H 4388 5450 30  0001 C CNN
+F 2 "Capacitors_SMD:C_0603" H 4388 5450 30  0001 C CNN
 F 3 "" H 4350 5600 60  0000 C CNN
 	1    4350 5600
@@
 F 0 "C6" H 3775 5700 50  0000 L CNN
 F 1 "10pF" H 3775 5500 50  0000 L CNN
-F 2 "_std:_0603" H 3788 5450 30  0001 C CNN
+F 2 "Capacitors_SMD:C_0603" H 3788 5450 30  0001 C CNN
 F 3 "" H 3750 5600 60  0000 C CNN
 	1    3750 5600
@@
 F 0 "C4" H 1775 1650 50  0000 L CNN
 F 1 "100nF" H 1775 1450 50  0000 L CNN
-F 2 "_std:_0603" H 1788 1400 30  0001 C CNN
+F 2 "Capacitors_SMD:C_0603" H 1788 1400 30  0001 C CNN
 F 3 "" H 1750 1550 60  0000 C CNN
 	1    1750 1550
@@
 L R R3
 U 1 1 55622F4C
-P 5550 1650
-F 0 "R3" V 5630 1650 50  0000 C CNN
-F 1 "1K" V 5550 1650 50  0000 C CNN
-F 2 "_std:_0603" V 5480 1650 30  0001 C CNN
-F 3 "" H 5550 1650 30  0000 C CNN
-	1    5550 1650
+P 5050 1650
+F 0 "R3" V 5130 1650 50  0000 C CNN
+F 1 "1K" V 5050 1650 50  0000 C CNN
+F 2 "Resistors_SMD:R_0603" V 4980 1650 30  0001 C CNN
+F 3 "" H 5050 1650 30  0000 C CNN
+	1    5050 1650
 	0    -1   -1   0
 $EndComp
@@
 L LED D1
 U 1 1 55624274
-P 5100 1350
-F 0 "D1" H 5100 1450 50  0000 C CNN
-F 1 "RX" H 5100 1250 50  0000 C CNN
-F 2 "_std:_0603" H 5100 1350 60  0001 C CNN
-F 3 "" H 5100 1350 60  0000 C CNN
-	1    5100 1350
-	1    0    0    -1
+P 5500 1350
+F 0 "D1" H 5500 1450 50  0000 C CNN
+F 1 "RX" H 5500 1250 50  0000 C CNN
+F 2 "LEDs:LED-0603" H 5500 1350 60  0001 C CNN
+F 3 "" H 5500 1350 60  0000 C CNN
+	1    5500 1350
+	-1   0    0    1
 $EndComp
 $Comp
 L R R2
 U 1 1 5562427A
-P 5550 1350
-F 0 "R2" V 5630 1350 50  0000 C CNN
-F 1 "1K" V 5550 1350 50  0000 C CNN
-F 2 "_std:_0603" V 5480 1350 30  0001 C CNN
-F 3 "" H 5550 1350 30  0000 C CNN
-	1    5550 1350
+P 5050 1350
+F 0 "R2" V 5130 1350 50  0000 C CNN
+F 1 "1K" V 5050 1350 50  0000 C CNN
+F 2 "Resistors_SMD:R_0603" V 4980 1350 30  0001 C CNN
+F 3 "" H 5050 1350 30  0000 C CNN
+	1    5050 1350
 	0    -1   -1   0
 $EndComp
@@
 L LED D2
 U 1 1 55622E77
-P 5100 1650
-F 0 "D2" H 5100 1750 50  0000 C CNN
-F 1 "TX" H 5100 1550 50  0000 C CNN
-F 2 "_std:_0603" H 5100 1650 60  0001 C CNN
-F 3 "" H 5100 1650 60  0000 C CNN
-	1    5100 1650
-	1    0    0    -1
+P 5500 1650
+F 0 "D2" H 5500 1750 50  0000 C CNN
+F 1 "TX" H 5500 1550 50  0000 C CNN
+F 2 "LEDs:LED-0603" H 5500 1650 60  0001 C CNN
+F 3 "" H 5500 1650 60  0000 C CNN
+	1    5500 1650
+	-1   0    0    1
 $EndComp
 Text Label 9950 4550 2    40   ~ 0
@@
 F 0 "C10" H 8875 1850 50  0000 L CNN
 F 1 "1uF" H 8875 1650 50  0000 L CNN
-F 2 "_std:_0603" H 8888 1600 30  0001 C CNN
+F 2 "Capacitors_SMD:C_0603" H 8888 1600 30  0001 C CNN
 F 3 "" H 8850 1750 60  0000 C CNN
 	1    8850 1750
@@
 F 0 "C12" H 9975 1850 50  0000 L CNN
 F 1 "1uF" H 9975 1650 50  0000 L CNN
-F 2 "_std:_0603" H 9988 1600 30  0001 C CNN
+F 2 "Capacitors_SMD:C_0603" H 9988 1600 30  0001 C CNN
 F 3 "" H 9950 1750 60  0000 C CNN
 	1    9950 1750
@@
 	1    0    0    -1
 $EndComp
-Text Notes 7400 7500 0    60   ~ 12
-nRF24 radio module
-Text Notes 10750 7650 0    60   ~ 12
-A
-Text Notes 8200 7650 0    60   ~ 0
-04.11.2015
-Text Notes 7050 7100 0    60   ~ 0
-Author: Michael Spieler
 $Comp
 L C C11
@@
 F 0 "C11" H 9800 2850 50  0000 L CNN
 F 1 "100nF" V 9600 2850 50  0000 L CNN
-F 2 "_std:_0603" H 9788 2800 30  0001 C CNN
+F 2 "Capacitors_SMD:C_0603" H 9788 2800 30  0001 C CNN
 F 3 "" H 9750 2950 60  0000 C CNN
 	1    9750 2950
@@
 F 0 "R4" V 9430 2950 50  0000 C CNN
 F 1 "1.5k" V 9350 2950 50  0000 C CNN
-F 2 "_std:_0603" V 9280 2950 30  0001 C CNN
+F 2 "Resistors_SMD:R_0603" V 9280 2950 30  0001 C CNN
 F 3 "" H 9350 2950 30  0000 C CNN
 	1    9350 2950
@@
 F 0 "C8" H 7575 4600 50  0000 L CNN
 F 1 "100nF" H 7575 4400 50  0000 L CNN
-F 2 "_std:_0603" H 7588 4350 30  0001 C CNN
+F 2 "Capacitors_SMD:C_0603" H 7588 4350 30  0001 C CNN
 F 3 "" H 7550 4500 60  0000 C CNN
 	1    7550 4500
@@
 F 0 "C9" H 8625 1850 50  0000 L CNN
 F 1 "22uF" H 8625 1650 50  0000 L CNN
-F 2 "_std:_0603" H 8638 1600 30  0001 C CNN
+F 2 "Capacitors_SMD:C_0603" H 8638 1600 30  0001 C CNN
 F 3 "" H 8600 1750 60  0000 C CNN
 	1    8600 1750
@@
 F 0 "U3" H 9650 1800 60  0000 C CNN
 F 1 "MCP1703" H 9350 1800 60  0000 C CNN
-F 2 "_std:_SOT23-3" H 9300 2050 60  0001 C CNN
+F 2 "_div:_MCP1703-SOT-23A" H 9300 2050 60  0001 C CNN
 F 3 "" H 9300 2050 60  0000 C CNN
 	1    9400 1600
@@
 NoConn ~ 3600 1400
 $Comp
-L VCC #PWR026
-U 1 1 56E424AB
-P 5800 1250
-F 0 "#PWR026" H 5800 1100 50  0001 C CNN
-F 1 "VCC" H 5800 1400 50  0000 C CNN
-F 2 "" H 5800 1250 50  0000 C CNN
-F 3 "" H 5800 1250 50  0000 C CNN
-	1    5800 1250
-	1    0    0    -1
-$EndComp
-Wire Wire Line
-	5800 1250 5800 1650
-Connection ~ 5800 1350
-Wire Wire Line
-	5400 1350 5300 1350
-Wire Wire Line
-	5400 1650 5300 1650
-$Comp
 L C C13
 U 1 1 56E76711
@@
 F 0 "C13" H 6775 3500 50  0000 L CNN
 F 1 "1uF" H 6775 3300 50  0000 L CNN
-F 2 "_std:_0603" H 6788 3250 30  0001 C CNN
+F 2 "Capacitors_SMD:C_0603" H 6788 3250 30  0001 C CNN
 F 3 "" H 6750 3400 60  0000 C CNN
 	1    6750 3400
@@
 Connection ~ 6750 3250
 $Comp
-L GND #PWR027
+L GND #PWR026
 U 1 1 56E76C2F
 P 6750 3550
-F 0 "#PWR027" H 6750 3300 50  0001 C CNN
+F 0 "#PWR026" H 6750 3300 50  0001 C CNN
 F 1 "GND" H 6750 3400 50  0000 C CNN
 F 2 "" H 6750 3550 50  0000 C CNN
@@
 	1    0    0    -1
 $EndComp
+Wire Wire Line
+	5800 1350 5800 1750
+$Comp
+L GND #PWR027
+U 1 1 57531D1B
+P 5800 1750
+F 0 "#PWR027" H 5800 1500 50  0001 C CNN
+F 1 "GND" H 5800 1600 50  0000 C CNN
+F 2 "" H 5800 1750 50  0000 C CNN
+F 3 "" H 5800 1750 50  0000 C CNN
+	1    5800 1750
+	1    0    0    -1
+$EndComp
+Connection ~ 5800 1650
+Wire Wire Line
+	5200 1650 5300 1650
+Wire Wire Line
+	5200 1350 5300 1350
 $EndSCHEMATC
